File: projeto-uselless-box/projeto-uselless-box.kicad_pcb (KiCad board)
At the start: 2 copper layers, 13 parts, among them J2 Conn_Para_Fita, J3 Conn_Para_PowerBank, M1 Motor_Servo-Edit, M2 Motor_Servo-Edit, M3 Motor_Servo-Edit, Q1 TIP41, SW1 SW_DPST_x2

Commit message: Minimal changes
Parts:
- R2: value 100R -> 80R

Commit message: Corections by Teacher A
Parts:
- moved M1 58.4 mm to (187.7, 132.5), turned to 90 degrees
- moved M2 47.0 mm to (196.2, 132.5), turned to 90 degrees
- moved M3 34.3 mm to (206.2, 132.5), turned to 90 degrees
- moved LS1 17.8 mm to (96.0, 129.3)
Routing:
- net +5V: track 398.7 -> 291.0 mm
- net GND: track 318.1 -> 373.9 mm
- net D5: track 105.3 -> 142.5 mm
- net D6: track 92.0 -> 126.1 mm
- net Net-(J1-SPK2): track 11.4 -> 29.2 mm
- net Net-(J1-SPK1): track 11.4 -> 29.2 mm
