File: projeto-uselless-box/projeto-uselless-box.kicad_pcb (KiCad board)
At the start: 2 copper layers, 100 x 79 mm, 16 parts, among them J2 Conn_Para_Fita, J3 Conn_Para_PowerBank, J4 Conn_01x01_Pin, J5 Conn_01x01_Pin, J6 Conn_01x01_Pin, M1 Motor_Servo-Edit, M2 Motor_Servo-Edit, M3 Motor_Servo-Edit, Q1 TIP41, SW1 SW_DPST_x2

Commit message: Minimal Details
Routing:
- net D5: track 130.5 -> 129.1 mm
- net D6: track 113.7 -> 112.3 mm
- net +5V: track 245.4 -> 244.0 mm
Changed lines of the file:
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@@
 	)
 	(segment
-		(start 91.54 136)
-		(end 87.54 132)
-		(width 1)
-		(layer "B.Cu")
-		(net 7)
-	)
-	(segment
-		(start 118 136)
-		(end 91.54 136)
+		(start 143 111)
+		(end 118 136)
 		(width 1)
 		(layer "B.Cu")
@@
 	)
 	(segment
-		(start 143 111)
-		(end 118 136)
-		(width 1)
-		(layer "B.Cu")
-		(net 7)
-	)
-	(segment
-		(start 87.54 132)
+		(start 118 136)
+		(end 94 136)
+		(width 1)
+		(layer "B.Cu")
+		(net 7)
+	)
+	(segment
+		(start 87.54 129.54)
 		(end 87.54 120.54)
 		(width 1)
@@
 	)
 	(segment
+		(start 94 136)
+		(end 87.54 129.54)
+		(width 1)
+		(layer "B.Cu")
+		(net 7)
+	)
+	(segment
 		(start 168.89 91.14)
 		(end 157 91.14)
@@
 	)
 	(segment
-		(start 83 98)
-		(end 83 130.46)
-		(width 1)
-		(layer "B.Cu")
-		(net 9)
-	)
-	(segment
 		(start 88.84 92.16)
 		(end 84.76 96.24)
@@
 	)
 	(segment
+		(start 83 98)
+		(end 83 128)
+		(width 1)
+		(layer "B.Cu")
+		(net 9)
+	)
+	(segment
+		(start 83 128)
+		(end 93 138)
+		(width 1)
+		(layer "B.Cu")
+		(net 9)
+	)
+	(segment
 		(start 167.46 124)
 		(end 153.46 138)
@@
 	)
 	(segment
-		(start 84.76 96.24)
-		(end 83 98)
-		(width 1)
-		(layer "B.Cu")
-		(net 9)
-	)
-	(segment
 		(start 167.46 119)
 		(end 149 137.46)
@@
 		(start 149 138)
 		(end 153.46 138)
-		(width 1)
-		(layer "B.Cu")
-		(net 9)
-	)
-	(segment
-		(start 83 130.46)
-		(end 90.54 138)
 		(width 1)
 		(layer "B.Cu")
@@
 	)
 	(segment
-		(start 90.54 138)
-		(end 143 138)
-		(width 1)
-		(layer "B.Cu")
-		(net 9)
-	)
-	(segment
 		(start 108.74 92.16)
 		(end 88.84 92.16)
@@
 	)
 	(segment
+		(start 84.76 96.24)
+		(end 83 98)
+		(width 1)
+		(layer "B.Cu")
+		(net 9)
+	)
+	(segment
 		(start 175 111.08)
 		(end 169.92 111.08)
@@
 	)
 	(segment
+		(start 93 138)
+		(end 143 138)
+		(width 1)
+		(layer "B.Cu")
+		(net 9)
+	)
+	(segment
 		(start 170.5 97)
 		(end 167.18 93.68)
@@
 	)
 	(segment
+		(start 108.74 87.08)
+		(end 106.08 87.08)
+		(width 1)
+		(layer "B.Cu")
+		(net 19)
+	)
+	(segment
 		(start 175 124)
 		(end 170 129)
@@
 	)
 	(segment
-		(start 108.74 87.08)
-		(end 106.08 87.08)
+		(start 105 86)
+		(end 105 66)
+		(width 1)
+		(layer "B.Cu")
+		(net 19)
+	)
+	(segment
+		(start 173 62)
+		(end 178 67)
+		(width 1)
+		(layer "B.Cu")
+		(net 19)
+	)
+	(segment
+		(start 170 124)
+		(end 175 124)
+		(width 1)
+		(layer "B.Cu")
+		(net 19)
+	)
+	(segment
+		(start 164 68)
+		(end 158 62)
+		(width 1)
+		(layer "B.Cu")
+		(net 19)
+	)
+	(segment
+		(start 178 114)
+		(end 178 116)
+		(width 1)
+		(layer "B.Cu")
+		(net 19)
+	)
+	(segment
+		(start 158 62)
+		(end 167.08 62)
+		(width 1)
+		(layer "B.Cu")
+		(net 19)
+	)
+	(segment
+		(start 100 82.38)
+		(end 100 71)
+		(width 1)
+		(layer "B.Cu")
+		(net 19)
+	)
+	(segment
+		(start 175.08 101)
+		(end 178 98.08)
+		(width 1)
+		(layer "B.Cu")
+		(net 19)
+	)
+	(segment
+		(start 174 68.92)
+		(end 167.08 62)
+		(width 1)
+		(layer "B.Cu")
+		(net 19)
+	)
+	(segment
+		(start 164 68.5)
+		(end 164 68)
+		(width 1)
+		(layer "B.Cu")
+		(net 19)
+	)
+	(segment
+		(start 105 66)
+		(end 109 62)
+		(width 1)
+		(layer "B.Cu")
+		(net 19)
+	)
+	(segment
+		(start 174 68.92)
+		(end 173.92 68.92)
 		(width 1)
 		(layer "B.Cu")
@@
 	)
 	(segment
-		(start 173 62)
-		(end 178 67)
-		(width 1)
-		(layer "B.Cu")
-		(net 19)
-	)
-	(segment
-		(start 170 124)
-		(end 175 124)
-		(width 1)
-		(layer "B.Cu")
-		(net 19)
-	)
-	(segment
-		(start 164 68)
-		(end 158 62)
-		(width 1)
-		(layer "B.Cu")
-		(net 19)
-	)
-	(segment
-		(start 178 114)
-		(end 178 116)
-		(width 1)
-		(layer "B.Cu")
-		(net 19)
-	)
-	(segment
-		(start 158 62)
-		(end 167.08 62)
-		(width 1)
-		(layer "B.Cu")
-		(net 19)
-	)
-	(segment
-		(start 100 82.38)
-		(end 100 71)
-		(width 1)
-		(layer "B.Cu")
-		(net 19)
-	)
-	(segment
-		(start 175.08 101)
-		(end 178 98.08)
-		(width 1)
-		(layer "B.Cu")
-		(net 19)
-	)
-	(segment
-		(start 174 68.92)
-		(end 167.08 62)
-		(width 1)
-		(layer "B.Cu")
-		(net 19)
-	)
-	(segment
-		(start 164 68.5)
-		(end 164 68)
-		(width 1)
-		(layer "B.Cu")
-		(net 19)
-	)
-	(segment
-		(start 105 66)
-		(end 109 62)
-		(width 1)
-		(layer "B.Cu")
-		(net 19)
-	)
-	(segment
-		(start 105 86)
-		(end 105 66)
-		(width 1)
-		(layer "B.Cu")
-		(net 19)
-	)
-	(segment
-		(start 174 68.92)
-		(end 173.92 68.92)
-		(width 1)
-		(layer "B.Cu")
-		(net 19)
-	)
-	(segment
 		(start 178 67)
 		(end 178 98.08)
@@
 	)
 	(segment
+		(start 89.84 100.16)
+		(end 89.84 128.84)
+		(width 1)
+		(layer "B.Cu")
+		(net 44)
+	)
+	(segment
+		(start 117 134)
+		(end 141 110)
+		(width 1)
+		(layer "B.Cu")
+		(net 44)
+	)
+	(segment
 		(start 141 95.46)
 		(end 157 79.46)
@@
 	)
 	(segment
-		(start 89.84 100.16)
-		(end 89.84 131.3)
+		(start 89.84 128.84)
+		(end 95 134)
 		(width 1)
 		(layer "B.Cu")
@@
 	)
 	(segment
-		(start 92.54 134)
+		(start 95 134)
 		(end 117 134)
 		(width 1)
 		(layer "B.Cu")
-		(net 44)
-	)
-	(segment
-		(start 89.84 131.3)
-		(end 92.54 134)
-		(width 1)
-		(layer "B.Cu")
-		(net 44)
-	)
-	(segment
-		(start 117 134)
-		(end 141 110)
-		(width 1)
-		(layer "B.Cu")
