File: projeto-uselless-box/projeto-uselless-box.kicad_sch (KiCad schematic)
At the start: 12 parts, among them M1 Motor_Servo, M2 Motor_Servo, M3 Motor_Servo, SW1 SW_DPST_x2, SW2 SW_DPST_x2, U1 L7809, U2 L7809

Commit message: Added motors to substitute the leds and sound
Parts:
- removed BT2: Battery_Cell, symbol Device:Battery_Cell
- removed D1: FITA_de_LED, symbol Device:LED
- removed SW2: SW_DPST_x2, symbol Switch:SW_DPST_x2
- removed U1, U2: L7809, symbol Regulator_Linear:L7809
- added M4: Fita de Led, symbol Motor:Motor_DC
- added M5: Auto Falante, symbol Motor:Motor_DC
- added Q1, Q2: BC337, Package_TO_SOT_THT:TO-92_Inline, symbol Transistor_BJT:BC337
- added R2, R3: R, symbol Device:R
- added U3: L7812, symbol Regulator_Linear:L7812
Connections:
- net +5V: now also M2.2 (+), M3.2 (+)
- net D6: now also R3.1
- net D7: now also R2.1
- net GND: now also M4.2 (-), M5.2 (-), U3.2 (GND)
- net IN1: now also U3.1 (IN)
- net OUT1: now also Q1.1 (C), Q2.1 (C), U3.3 (OUT)
- new net: Q1.2 (B), R2.2
- new net: Q2.2 (B), R3.2
- new net: M5.1 (+), Q2.3 (E)
- new net: M4.1 (+), Q1.3 (E)

Commit message: Editing schematic
Parts:
- removed M5: Auto Falante, symbol Motor:Motor_DC
- removed Q2: BC337, Package_TO_SOT_THT:TO-92_Inline, symbol Transistor_BJT:BC337
- removed R3: R, symbol Device:R
Connections:
- net D7: no longer R2.1
- net D8: now also R2.1; no longer M1.1 (PWM)
- net D9: now reaches A1.24 (D9)
- net D9: now also M1.1 (PWM)
Other:
- moved on the sheet: M4, Q1, R2

Commit message: Fixing some things
Parts:
- removed BT1: Battery_Cell, symbol Device:Battery_Cell
- removed M1, M2, M3: Motor_Servo, symbol Motor:Motor_Servo
- removed M4: Fita de Led, symbol Motor:Motor_DC
- removed Q1: BC337, Package_TO_SOT_THT:TO-92_Inline, symbol Transistor_BJT:BC337
- removed U3: L7812, symbol Regulator_Linear:L7812
- added J1: ~, Arduino_Nano:DFPlayer, symbol Arduino_Nano:DFPlayer
- added J2: Conn_Para_Fita, TerminalBlock_Phoenix:TerminalBlock_Phoenix_MKDS-1,5-2-5.08_1x02_P5.08mm_Horizontal, symbol Connector:Conn_01x02_Pin
- added J3: Conn_Para_PowerBank, TerminalBlock_Phoenix:TerminalBlock_Phoenix_MKDS-1,5-2-5.08_1x02_P5.08mm_Horizontal, symbol Connector:Conn_01x02_Pin
- added LS1: Speaker, TerminalBlock_Phoenix:TerminalBlock_Phoenix_MKDS-1,5-2-5.08_1x02_P5.08mm_Horizontal, symbol Device:Speaker
- added M1, M2, M3: Motor_Servo-Edit, Connector_PinSocket_2.54mm:PinSocket_1x02_P2.54mm_Vertical, symbol New_Library:Motor_Servo-Edit
- added Q1: TIP41, Package_TO_SOT_THT:TO-220-3_Vertical, symbol Transistor_BJT:TIP41
- added R3: 1kR, Resistor_THT:R_Axial_DIN0207_L6.3mm_D2.5mm_P10.16mm_Horizontal, symbol Device:R
- R1: value R -> 10kR; footprint (none) -> Resistor_THT:R_Axial_DIN0207_L6.3mm_D2.5mm_P10.16mm_Horizontal
- R2: value R -> 100R; footprint (none) -> Resistor_THT:R_Axial_DIN0207_L6.3mm_D2.5mm_P10.16mm_Horizontal
- SW1: footprint (none) -> TerminalBlock_Phoenix:TerminalBlock_Phoenix_MKDS-1,5-2-5.08_1x02_P5.08mm_Horizontal
Connections:
- net +5V: now also J1.1 (VCC), M1.2 (+), M2.2 (+), M3.2 (+)
- net D10: now also M2.3 (PWM)
- net D11: now also M3.3 (PWM)
- net D6: now also R3.2
- net D9: now also M1.3 (PWM)
- net GND: now also J1.10 (GND), J3.1 (Pin_1), M1.1 (-), M2.1 (-), M3.1 (-), Q1.3 (E)
- net at R2.2: now also Q1.1 (B)
- net D5: now reaches A1.20 (D5)
- net D5: now also J1.3 (TX)
- net D7: no longer names the net of A1.22 (D7)
- new net: J1.2 (RX), R3.1
- new net: J1.8 (SPK1), LS1.1
- new net: J1.6 (SPK2), LS1.2
- new net: J2.2 (Pin_2), Q1.2 (C)
- new net: J2.1 (Pin_1), J3.2 (Pin_2)
Other:
- moved on the sheet: R1, SW1A

Commit message: Minimal changes
Parts:
- R2: value 100R -> 80R
Other:
- moved on the sheet: A1
Changed lines of the file:
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@@
 	(wire
 		(pts
-			(xy 76.2 62.23) (xy 72.39 62.23)
+			(xy 78.74 72.39) (xy 74.93 72.39)
 		)
 		(stroke
@@
 	(wire
 		(pts
-			(xy 76.2 69.85) (xy 72.39 69.85)
-		)
-		(stroke
-			(width 0)
-			(type default)
-		)
-	)
-	(wire
-		(pts
-			(xy 76.2 72.39) (xy 72.39 72.39)
+			(xy 78.74 80.01) (xy 74.93 80.01)
+		)
+		(stroke
+			(width 0)
+			(type default)
+		)
+	)
+	(wire
+		(pts
+			(xy 78.74 82.55) (xy 74.93 82.55)
 		)
 		(stroke
@@
 	(wire
 		(pts
-			(xy 54.61 33.02) (xy 54.61 36.83)
+			(xy 57.15 43.18) (xy 57.15 46.99)
 		)
 		(stroke
@@
 	(wire
 		(pts
-			(xy 57.15 93.98) (xy 57.15 90.17)
+			(xy 59.69 104.14) (xy 59.69 100.33)
 		)
 		(stroke
@@
 	(wire
 		(pts
-			(xy 76.2 67.31) (xy 72.39 67.31)
-		)
-		(stroke
-			(width 0)
-			(type default)
-		)
-	)
-	(wire
-		(pts
-			(xy 72.39 59.69) (xy 76.2 59.69)
-		)
-		(stroke
-			(width 0)
-			(type default)
-		)
-	)
-	(wire
-		(pts
-			(xy 76.2 77.47) (xy 72.39 77.47)
-		)
-		(stroke
-			(width 0)
-			(type default)
-		)
-	)
-	(wire
-		(pts
-			(xy 76.2 74.93) (xy 72.39 74.93)
+			(xy 78.74 77.47) (xy 74.93 77.47)
+		)
+		(stroke
+			(width 0)
+			(type default)
+		)
+	)
+	(wire
+		(pts
+			(xy 74.93 69.85) (xy 78.74 69.85)
+		)
+		(stroke
+			(width 0)
+			(type default)
+		)
+	)
+	(wire
+		(pts
+			(xy 78.74 87.63) (xy 74.93 87.63)
+		)
+		(stroke
+			(width 0)
+			(type default)
+		)
+	)
+	(wire
+		(pts
+			(xy 78.74 85.09) (xy 74.93 85.09)
 		)
 		(stroke
@@
 	(global_label "D11"
 		(shape input)
-		(at 76.2 74.93 0)
+		(at 78.74 85.09 0)
 		(fields_autoplaced yes)
 		(effects
@@
 		)
 		(property "Intersheetrefs" "${INTERSHEET_REFS}"
-			(at 82.8742 74.93 0)
+			(at 85.4142 85.09 0)
 			(effects
 				(font
@@
 	(global_label "D8"
 		(shape input)
-		(at 76.2 67.31 0)
+		(at 78.74 77.47 0)
 		(fields_autoplaced yes)
 		(effects
@@
 		)
 		(property "Intersheetrefs" "${INTERSHEET_REFS}"
-			(at 81.6647 67.31 0)
+			(at 84.2047 77.47 0)
 			(effects
 				(font
@@
 	(global_label "D12"
 		(shape input)
-		(at 76.2 77.47 0)
+		(at 78.74 87.63 0)
 		(fields_autoplaced yes)
 		(effects
@@
 		)
 		(property "Intersheetrefs" "${INTERSHEET_REFS}"
-			(at 82.8742 77.47 0)
+			(at 85.4142 87.63 0)
 			(effects
 				(font
@@
 	(global_label "D6"
 		(shape input)
-		(at 76.2 62.23 0)
+		(at 78.74 72.39 0)
 		(fields_autoplaced yes)
 		(effects
@@
 		)
 		(property "Intersheetrefs" "${INTERSHEET_REFS}"
-			(at 81.6647 62.23 0)
+			(at 84.2047 72.39 0)
 			(effects
 				(font
@@
 	(global_label "D9"
 		(shape input)
-		(at 76.2 69.85 0)
+		(at 78.74 80.01 0)
 		(fields_autoplaced yes)
 		(effects
@@
 		)
 		(property "Intersheetrefs" "${INTERSHEET_REFS}"
-			(at 81.6647 69.85 0)
+			(at 84.2047 80.01 0)
 			(effects
 				(font
@@
 	(global_label "D5"
 		(shape input)
-		(at 76.2 59.69 0)
+		(at 78.74 69.85 0)
 		(fields_autoplaced yes)
 		(effects
@@
 		)
 		(property "Intersheetrefs" "${INTERSHEET_REFS}"
-			(at 81.6647 59.69 0)
+			(at 84.2047 69.85 0)
 			(effects
 				(font
@@
 	(global_label "D10"
 		(shape input)
-		(at 76.2 72.39 0)
+		(at 78.74 82.55 0)
 		(fields_autoplaced yes)
 		(effects
@@
 		)
 		(property "Intersheetrefs" "${INTERSHEET_REFS}"
-			(at 82.8742 72.39 0)
+			(at 85.4142 82.55 0)
 			(effects
 				(font
@@
 	(symbol
 		(lib_id "MCU_Module:Arduino_UNO_R3")
-		(at 59.69 62.23 0)
+		(at 62.23 72.39 0)
 		(mirror y)
 		(unit 1)
@@
 		(fields_autoplaced yes)
 		(property "Reference" "A1"
-			(at 65.3481 92.71 0)
+			(at 67.8881 102.87 0)
 			(effects
 				(font
@@
 		)
 		(property "Value" "Arduino_UNO_R3"
-			(at 65.3481 90.17 0)
+			(at 67.8881 100.33 0)
 			(effects
 				(font
@@
 		)
 		(property "Footprint" "Module:Arduino_UNO_R3"
-			(at 59.69 62.23 0)
+			(at 62.23 72.39 0)
 			(effects
 				(font
@@
 		)
 		(property "Datasheet" "https://www.arduino.cc/en/Main/arduinoBoardUno"
-			(at 59.69 62.23 0)
+			(at 62.23 72.39 0)
 			(effects
 				(font
@@
 		)
 		(property "Description" "Arduino UNO Microcontroller Module, release 3"
-			(at 59.69 62.23 0)
+			(at 62.23 72.39 0)
 			(effects
 				(font
@@
 			)
 		)
-		(property "Value" "100R"
+		(property "Value" "80R"
 			(at 129.54 92.71 90)
 			(effects
@@
 	(symbol
 		(lib_id "power:GND")
-		(at 57.15 93.98 0)
+		(at 59.69 104.14 0)
 		(mirror y)
 		(unit 1)
@@
 		(fields_autoplaced yes)
 		(property "Reference" "#PWR02"
-			(at 57.15 100.33 0)
+			(at 59.69 110.49 0)
 			(effects
 				(font
@@
 		)
 		(property "Value" "GND"
-			(at 57.15 99.06 0)
+			(at 59.69 109.22 0)
 			(effects
 				(font
@@
 		)
 		(property "Footprint" ""
-			(at 57.15 93.98 0)
+			(at 59.69 104.14 0)
 			(effects
 				(font
@@
 		)
 		(property "Datasheet" ""
-			(at 57.15 93.98 0)
+			(at 59.69 104.14 0)
 			(effects
 				(font
@@
 		)
 		(property "Description" "Power symbol creates a global label with name \"GND\" , ground"
-			(at 57.15 93.98 0)
+			(at 59.69 104.14 0)
 			(effects
 				(font
@@
 	(symbol
 		(lib_id "power:+5V")
-		(at 54.61 33.02 0)
+		(at 57.15 43.18 0)
 		(mirror y)
 		(unit 1)
@@
 		(fields_autoplaced yes)
 		(property "Reference" "#PWR01"
-			(at 54.61 36.83 0)
+			(at 57.15 46.99 0)
 			(effects
 				(font
@@
 		)
 		(property "Value" "+5V"
-			(at 54.61 27.94 0)
+			(at 57.15 38.1 0)
 			(effects
 				(font
@@
 		)
 		(property "Footprint" ""
-			(at 54.61 33.02 0)
+			(at 57.15 43.18 0)
 			(effects
 				(font
@@
 		)
 		(property "Datasheet" ""
-			(at 54.61 33.02 0)
+			(at 57.15 43.18 0)
 			(effects
 				(font
@@
 		)
 		(property "Description" "Power symbol creates a global label with name \"+5V\""
-			(at 54.61 33.02 0)
-			(effects
-				(font
+			(at 57.15 43.18 0)
+			(effects
+				(font

Commit message: ShortedA
Parts:
- added J4, J5, J6: Conn_01x01_Pin, Connector_PinSocket_2.54mm:PinSocket_1x01_P2.54mm_Vertical, symbol Connector:Conn_01x01_Pin
Connections:
- net D10: now also J5.1 (Pin_1); no longer M2.3 (PWM)
- net D11: now also J6.1 (Pin_1); no longer M3.3 (PWM)
- net D9: now also J4.1 (Pin_1); no longer M1.3 (PWM)
Other:
- moved on the sheet: J1, LS1, R3
